Commit message: [feat] Add RG2 gripper support in MoveIt configuration and related files

File: xarm_moveit_config/srdf/_uf850_macro.srdf.xacro (robot description, xacro)
@@ -10,5 +10,5 @@
   <!-- SUBGROUPS: Groups can also be formed by referencing to already defined group names -->
   <xacro:macro name="uf850_macro_srdf" params="prefix=''
-    add_gripper='false' add_vacuum_gripper='false' add_bio_gripper='false' add_other_geometry='false' ">
+    add_gripper='false' add_vacuum_gripper='false' add_bio_gripper='false' add_rg2_gripper='false' add_other_geometry='false' ">
     <group name="${prefix}uf850">
       <joint name="${prefix}world_joint" />
@@ -33,5 +33,8 @@
         <joint name="${prefix}joint_tcp" />
       </xacro:if>
-      <xacro:if value="${not add_gripper and not add_bio_gripper and not add_vacuum_gripper and add_other_geometry}">
+      <xacro:if value="${not add_gripper and not add_bio_gripper and not add_vacuum_gripper and add_rg2_gripper}">
+        <joint name="${prefix}joint0" />
+      </xacro:if>
+      <xacro:if value="${not add_gripper and not add_bio_gripper and not add_vacuum_gripper and not add_rg2_gripper and add_other_geometry}">
         <joint name="${prefix}other_geometry_fix" />
         <joint name="${prefix}joint_tcp" />
@@ -178,6 +181,91 @@
       <disable_collisions link1="${prefix}link_eef" link2="${prefix}xarm_vacuum_gripper_link" reason="Adjacent" />
     </xacro:if>
+    <!-- RG2 gripper -->
+    <xacro:if value="${not add_gripper and not add_bio_gripper and not add_vacuum_gripper and add_rg2_gripper}">
+      <group name="${prefix}rg2_gripper">
+        <link name="${prefix}rg2_base_link" />
+        <link name="${prefix}rg2_left_outer_knuckle" />
+        <link name="${prefix}rg2_left_inner_knuckle" />
+        <link name="${prefix}rg2_left_inner_finger" />
+        <link name="${prefix}rg2_right_outer_knuckle" />
+        <link name="${prefix}rg2_right_inner_knuckle" />
+        <link name="${prefix}rg2_right_inner_finger" />
+        <joint name="${prefix}rg2_finger_joint" />
+      </group>
+      <group_state name="open" group="${prefix}rg2_gripper">
+        <joint name="${prefix}rg2_finger_joint" value="0.785398" />
+      </group_state>
+      <group_state name="close" group="${prefix}rg2_gripper">
+        <joint name="${prefix}rg2_finger_joint" value="-0.558505" />
+      </group_state>
+      <!-- END EFFECTOR -->
+      <end_effector name="${prefix}rg2_gripper" parent_link="${prefix}link_eef" group="${prefix}rg2_gripper" />
+      <!-- PASSIVE JOINTS -->
+      <passive_joint name="${prefix}joint0" />
+      <passive_joint name="${prefix}rg2_left_inner_knuckle_joint" />
+      <passive_joint name="${prefix}rg2_left_inner_finger_joint" />
+      <passive_joint name="${prefix}rg2_right_outer_knuckle_joint" />
+      <passive_joint name="${prefix}rg2_right_inner_knuckle_joint" />
+      <passive_joint name="${prefix}rg2_right_inner_finger_joint" />
+      <!-- DISABLE COLLISIONS -->
+      <disable_collisions link1="${prefix}rg2_base_link" link2="${prefix}link6" reason="Adjacent" />
+      <disable_collisions link1="${prefix}rg2_base_link" link2="${prefix}link_eef" reason="Adjacent" />
+      <disable_collisions link1="${prefix}rg2_base_link" link2="${prefix}rg2_left_outer_knuckle" reason="Adjacent" />
+      <disable_collisions link1="${prefix}rg2_base_link" link2="${prefix}rg2_right_outer_knuckle" reason="Adjacent" />
+      <disable_collisions link1="${prefix}rg2_base_link" link2="${prefix}rg2_left_inner_knuckle" reason="Adjacent" />
+      <disable_collisions link1="${prefix}rg2_base_link" link2="${prefix}rg2_right_inner_knuckle" reason="Adjacent" />
+      <disable_collisions link1="${prefix}rg2_base_link" link2="${prefix}rg2_left_inner_finger" reason="Never" />
+      <disable_collisions link1="${prefix}rg2_base_link" link2="${prefix}rg2_right_inner_finger" reason="Never" />
+      <disable_collisions link1="${prefix}rg2_left_outer_knuckle" link2="${prefix}rg2_left_inner_knuckle" reason="Never" />
+      <disable_collisions link1="${prefix}rg2_left_outer_knuckle" link2="${prefix}rg2_left_inner_finger" reason="Adjacent" />
+      <disable_collisions link1="${prefix}rg2_left_outer_knuckle" link2="${prefix}rg2_right_outer_knuckle" reason="Never" />
+      <disable_collisions link1="${prefix}rg2_left_outer_knuckle" link2="${prefix}rg2_right_inner_knuckle" reason="Never" />
+      <disable_collisions link1="${prefix}rg2_left_outer_knuckle" link2="${prefix}rg2_right_inner_finger" reason="Never" />
+      <disable_collisions link1="${prefix}rg2_left_inner_knuckle" link2="${prefix}rg2_left_inner_finger" reason="Default" />
+      <disable_collisions link1="${prefix}rg2_left_inner_knuckle" link2="${prefix}rg2_right_outer_knuckle" reason="Never" />
+      <disable_collisions link1="${prefix}rg2_left_inner_knuckle" link2="${prefix}rg2_right_inner_knuckle" reason="Never" />
+      <disable_collisions link1="${prefix}rg2_left_inner_knuckle" link2="${prefix}rg2_right_inner_finger" reason="Never" />
+      <disable_collisions link1="${prefix}rg2_left_inner_finger" link2="${prefix}rg2_right_outer_knuckle" reason="Never" />
+      <disable_collisions link1="${prefix}rg2_left_inner_finger" link2="${prefix}rg2_right_inner_knuckle" reason="Never" />
+      <disable_collisions link1="${prefix}rg2_right_outer_knuckle" link2="${prefix}rg2_right_inner_knuckle" reason="Never" />
+      <disable_collisions link1="${prefix}rg2_right_outer_knuckle" link2="${prefix}rg2_right_inner_finger" reason="Adjacent" />
+      <disable_collisions link1="${prefix}rg2_right_inner_knuckle" link2="${prefix}rg2_right_inner_finger" reason="Default" />
+      <disable_collisions link1="${prefix}rg2_left_inner_finger" link2="${prefix}rg2_right_inner_finger" reason="Never" />
+      <disable_collisions link1="${prefix}link3" link2="${prefix}rg2_base_link" reason="Never" />
+      <disable_collisions link1="${prefix}link3" link2="${prefix}rg2_left_outer_knuckle" reason="Never" />
+      <disable_collisions link1="${prefix}link3" link2="${prefix}rg2_right_outer_knuckle" reason="Never" />
+      <disable_collisions link1="${prefix}link3" link2="${prefix}rg2_left_inner_knuckle" reason="Never" />
+      <disable_collisions link1="${prefix}link3" link2="${prefix}rg2_right_inner_knuckle" reason="Never" />
+      <disable_collisions link1="${prefix}link3" link2="${prefix}rg2_left_inner_finger" reason="Never" />
+      <disable_collisions link1="${prefix}link3" link2="${prefix}rg2_right_inner_finger" reason="Never" />
+      <disable_collisions link1="${prefix}link4" link2="${prefix}rg2_base_link" reason="Never" />
+      <disable_collisions link1="${prefix}link4" link2="${prefix}rg2_left_outer_knuckle" reason="Never" />
+      <disable_collisions link1="${prefix}link4" link2="${prefix}rg2_right_outer_knuckle" reason="Never" />
+      <disable_collisions link1="${prefix}link4" link2="${prefix}rg2_left_inner_knuckle" reason="Never" />
+      <disable_collisions link1="${prefix}link4" link2="${prefix}rg2_right_inner_knuckle" reason="Never" />
+      <disable_collisions link1="${prefix}link4" link2="${prefix}rg2_left_inner_finger" reason="Never" />
+      <disable_collisions link1="${prefix}link4" link2="${prefix}rg2_right_inner_finger" reason="Never" />
+      <disable_collisions link1="${prefix}link5" link2="${prefix}rg2_base_link" reason="Never" />
+      <disable_collisions link1="${prefix}link5" link2="${prefix}rg2_left_outer_knuckle" reason="Never" />
+      <disable_collisions link1="${prefix}link5" link2="${prefix}rg2_right_outer_knuckle" reason="Never" />
+      <disable_collisions link1="${prefix}link5" link2="${prefix}rg2_left_inner_knuckle" reason="Never" />
+      <disable_collisions link1="${prefix}link5" link2="${prefix}rg2_right_inner_knuckle" reason="Never" />
+      <disable_collisions link1="${prefix}link5" link2="${prefix}rg2_left_inner_finger" reason="Never" />
+      <disable_collisions link1="${prefix}link5" link2="${prefix}rg2_right_inner_finger" reason="Never" />
+      <disable_collisions link1="${prefix}link6" link2="${prefix}rg2_left_outer_knuckle" reason="Never" />
+      <disable_collisions link1="${prefix}link6" link2="${prefix}rg2_right_outer_knuckle" reason="Never" />
+      <disable_collisions link1="${prefix}link6" link2="${prefix}rg2_left_inner_knuckle" reason="Never" />
+      <disable_collisions link1="${prefix}link6" link2="${prefix}rg2_right_inner_knuckle" reason="Never" />
+      <disable_collisions link1="${prefix}link6" link2="${prefix}rg2_left_inner_finger" reason="Never" />
+      <disable_collisions link1="${prefix}link6" link2="${prefix}rg2_right_inner_finger" reason="Never" />
+      <disable_collisions link1="${prefix}link_eef" link2="${prefix}rg2_left_outer_knuckle" reason="Never" />
+      <disable_collisions link1="${prefix}link_eef" link2="${prefix}rg2_right_outer_knuckle" reason="Never" />
+      <disable_collisions link1="${prefix}link_eef" link2="${prefix}rg2_left_inner_knuckle" reason="Never" />
+      <disable_collisions link1="${prefix}link_eef" link2="${prefix}rg2_right_inner_knuckle" reason="Never" />
+      <disable_collisions link1="${prefix}link_eef" link2="${prefix}rg2_left_inner_finger" reason="Never" />
+      <disable_collisions link1="${prefix}link_eef" link2="${prefix}rg2_right_inner_finger" reason="Never" />
+    </xacro:if>
     <!-- other box -->
-    <xacro:if value="${not add_gripper and not add_bio_gripper and not add_vacuum_gripper and add_other_geometry}">
+    <xacro:if value="${not add_gripper and not add_bio_gripper and not add_vacuum_gripper and not add_rg2_gripper and add_other_geometry}">
       <!-- <group name="${prefix}other_geometry">
         <joint name="${prefix}other_geometry_fix" />

File: xarm_moveit_config/srdf/xarm.srdf.xacro (robot description, xacro)
@@ -8,7 +8,8 @@
   <xacro:arg name="add_vacuum_gripper" default="false" />
   <xacro:arg name="add_bio_gripper" default="false" />
+  <xacro:arg name="add_rg2_gripper" default="false" />
   <xacro:arg name="add_other_geometry" default="false" />
   <xacro:include filename="$(find xarm_moveit_config)/srdf/xarm_macro.srdf.xacro" />
   <xacro:xarm_macro_srdf prefix="$(arg prefix)" dof="$(arg dof)" robot_type="$(arg robot_type)"
-    add_gripper="$(arg add_gripper)" add_vacuum_gripper="$(arg add_vacuum_gripper)" add_bio_gripper="$(arg add_bio_gripper)" add_other_geometry="$(arg add_other_geometry)" />
+    add_gripper="$(arg add_gripper)" add_vacuum_gripper="$(arg add_vacuum_gripper)" add_bio_gripper="$(arg add_bio_gripper)" add_rg2_gripper="$(arg add_rg2_gripper)" add_other_geometry="$(arg add_other_geometry)" />
 </robot>

File: xarm_moveit_config/srdf/xarm_macro.srdf.xacro (robot description, xacro)
@@ -2,5 +2,5 @@
 <robot xmlns:xacro="http://wiki.ros.org/xacro" name="xarm_srdf">
   <xacro:macro name="xarm_macro_srdf" params="prefix:='' dof:=7 robot_type:='xarm'
-    add_gripper:='false' add_vacuum_gripper:='false' add_bio_gripper:='false' add_other_geometry:='false' ">
+    add_gripper:='false' add_vacuum_gripper:='false' add_bio_gripper:='false' add_rg2_gripper:='false' add_other_geometry:='false' ">
     <xacro:if value="${dof == 5}">
       <xacro:include filename="$(find xarm_moveit_config)/srdf/_xarm5_macro.srdf.xacro" />
@@ -12,5 +12,5 @@
         <xacro:include filename="$(find xarm_moveit_config)/srdf/_uf850_macro.srdf.xacro" />
         <xacro:uf850_macro_srdf prefix="${prefix}"
-          add_gripper="${add_gripper}" add_vacuum_gripper="${add_vacuum_gripper}" add_bio_gripper="${add_bio_gripper}" add_other_geometry="${add_other_geometry}"  />
+          add_gripper="${add_gripper}" add_vacuum_gripper="${add_vacuum_gripper}" add_bio_gripper="${add_bio_gripper}" add_rg2_gripper="${add_rg2_gripper}" add_other_geometry="${add_other_geometry}"  />
       </xacro:if>
       <xacro:if value="${robot_type == 'lite'}">
