Commit message: feat(xarm_controller): restore joint-space command interfaces behind joint_mode
joint1..6 have been state-only since Cartesian tcp/ft support replaced this
hardware component's original joint-servo implementation: the arm runs in
XARM_MODE::POSE for its whole lifetime and is commanded through the tcp gpio
with set_position(), so no controller can move it per joint (a
JointGroupPositionController or joint_trajectory_controller has nothing to
claim). That original implementation still exists on this fork's own humble
branch, predating the Cartesian rework -- this ports it forward as an
opt-in, launch-time-only mode rather than reimplementing it from scratch.

joint_mode:=true (default false, today's behavior unchanged):
- exports joint1..6 position+velocity command interfaces instead of the tcp
  and ft gpio blocks, and skips the ft_sensor block entirely
- runs the arm in XARM_MODE::SERVO (or VELO_JOINT if velocity_control is
  also set) instead of XARM_MODE::POSE
- write() dispatches to set_servo_angle_j()/vc_set_joint_velocity() instead
  of set_position(), restoring humble's own throttled-send logic
- skips homing and force control entirely -- neither is compatible with
  SERVO/VELO_JOINT mode, and this mode never armed either in the first place

These are mutually exclusive by construction, not a live toggle: the arm can
only be in one XARM_MODE at a time, so on_init() requires the URDF to
declare exactly the interface set the chosen mode needs (joints only, or
gpios+sensor only), and rejects a mismatch rather than silently ignoring it.

Compiles clean; the default (joint_mode:=false) path is unchanged and its
existing xacro-render tests in the mmr-robot repo still pass. Not yet
exercised against a real arm or a controller actually driving the new joint
interfaces -- that needs bench validation before this goes anywhere near
main.

File: xarm_description/urdf/uf850/uf850.ros2_control.xacro (robot description, xacro)
@@ -3,4 +3,5 @@
   <xacro:macro name="uf850_ros2_control" params="prefix
     velocity_control:='false'
+    joint_mode:='false'
     ros2_control_plugin:='uf_robot_hardware/UFRobotSystemHardware'
     hw_ns:='xarm' add_gripper:='false' add_bio_gripper:='false'
@@ -30,4 +31,12 @@
           <param name="hw_ns">${prefix}${hw_ns}</param>
           <param name="velocity_control">${velocity_control}</param>
+          <!-- true: joints get position+velocity command interfaces and the arm is
+               commanded with set_servo_angle_j()/vc_set_joint_velocity() in
+               XARM_MODE::SERVO or VELO_JOINT, the same way this hardware component did
+               before Cartesian tcp/ft support replaced it. Mutually exclusive with that
+               support, since the arm can only be in one XARM_MODE at a time, not a
+               launch-time choice to layer both onto one running arm. false (default):
+               today's Cartesian tcp/ft gpio behaviour, XARM_MODE::POSE, unchanged. -->
+          <param name="joint_mode">${joint_mode}</param>
           <param name="prefix">P${prefix}</param>
           <param name="robot_ip">R${robot_ip}</param>
@@ -84,4 +93,8 @@
       </hardware>
       <joint name="${prefix}joint1">
+        <xacro:if value="${joint_mode}">
+          <command_interface name="position"/>
+          <command_interface name="velocity"/>
+        </xacro:if>
         <state_interface name="position">
           <param name="initial_value">0.0</param>
@@ -93,4 +106,8 @@
       </joint>
       <joint name="${prefix}joint2">
+        <xacro:if value="${joint_mode}">
+          <command_interface name="position"/>
+          <command_interface name="velocity"/>
+        </xacro:if>
         <state_interface name="position">
           <param name="initial_value">0.0</param>
@@ -102,4 +119,8 @@
       </joint>
       <joint name="${prefix}joint3">
+        <xacro:if value="${joint_mode}">
+          <command_interface name="position"/>
+          <command_interface name="velocity"/>
+        </xacro:if>
         <state_interface name="position">
           <param name="initial_value">0.0</param>
@@ -111,4 +132,8 @@
       </joint>
       <joint name="${prefix}joint4">
+        <xacro:if value="${joint_mode}">
+          <command_interface name="position"/>
+          <command_interface name="velocity"/>
+        </xacro:if>
         <state_interface name="position">
           <param name="initial_value">0.0</param>
@@ -120,4 +145,8 @@
       </joint>
       <joint name="${prefix}joint5">
+        <xacro:if value="${joint_mode}">
+          <command_interface name="position"/>
+          <command_interface name="velocity"/>
+        </xacro:if>
         <state_interface name="position">
           <param name="initial_value">0.0</param>
@@ -129,15 +158,21 @@
       </joint>
       <joint name="${prefix}joint6">
-        <state_interface name="position">
-          <param name="initial_value">0.0</param>
-        </state_interface>
-        <state_interface name="velocity">
-          <param name="initial_value">0.0</param>
-        </state_interface>
-        <!-- <state_interface name="effort"/> -->
-      </joint>
-      <!-- Cartesian TCP command and state, SI units (m, rad). The arm runs in
-           XARM_MODE::POSE for its whole lifetime, so motion is commanded with
-           set_position() through these interfaces rather than per joint. -->
+        <xacro:if value="${joint_mode}">
+          <command_interface name="position"/>
+          <command_interface name="velocity"/>
+        </xacro:if>
+        <state_interface name="position">
+          <param name="initial_value">0.0</param>
+        </state_interface>
+        <state_interface name="velocity">
+          <param name="initial_value">0.0</param>
+        </state_interface>
+        <!-- <state_interface name="effort"/> -->
+      </joint>
+      <!-- Cartesian TCP command and state, SI units (m, rad), and the force control gpios
+           below: all three are POSE-mode only, so joint_mode drops them entirely rather
+           than declaring interfaces the hardware component won't export in that mode
+           (its on_init() requires zero gpios/sensors when joint_mode is set, to match). -->
+      <xacro:unless value="${joint_mode}">
       <gpio name="${prefix}tcp">
         <command_interface name="x"/>
@@ -228,4 +263,5 @@
         </state_interface>
       </sensor>
+      </xacro:unless>
     </ros2_control>
   </xacro:macro>
